File: led-strip-connector/led-strip-connector-backups/led-strip-connector.kicad_sch (KiCad schematic)
At the start: 15 parts, among them J1 Conn_01x03_Pin, Q1 UMH3N, U2 ESP-12F, U3 LM1117MP-3.3, U4 CH340C

Commit message: new pcb
Parts:
- removed U4: CH340C, Package_SO:SOIC-16_3.9x9.9mm_P1.27mm, symbol Interface_USB:CH340C
- added C1: 100n, Capacitor_SMD:C_0603_1608Metric, symbol Device:C_Small
- added C3: 10u, Capacitor_SMD:C_1206_3216Metric, symbol Device:C_Small
- added D1, D2: LED, LED_SMD:LED_1206_3216Metric, symbol Device:LED
- added R2, R3: 100, Resistor_SMD:R_0603_1608Metric, symbol Device:R
- added U1: FT232RNL, Package_SO:SSOP-28_5.3x10.2mm_P0.65mm, symbol Interface_USB:FT232RL
- C2: renamed from C1; LCSC Part Number C282519 -> (none)
- C4: renamed from C2; LCSC Part Number C282519 -> (none)
- C5: renamed from C3; LCSC Part Number C19110 -> (none)
- C6: renamed from C4; LCSC Part Number C19110 -> (none)
- J1: LCSC Part Number C157929 -> (none)
- Q1: LCSC Part Number C62892 -> (none)
- R1: LCSC Part Number C105881 -> (none)
- R4: renamed from R2; LCSC Part Number C98220 -> (none)
- R5: renamed from R3; LCSC Part Number C98220 -> (none)
- R7: renamed from R4; LCSC Part Number C105580 -> (none)
- R8: renamed from R5; LCSC Part Number C105580 -> (none)
- U2: LCSC Part Number C82891 -> (none)
- U3: LCSC Part Number C498153 -> (none)
- USB1: value C31-M12 -> USB4105-GF-A; footprint Connector_USB:USB_C_Receptacle_HRO_TYPE-C-31-M-12 -> Connector_USB:USB_C_Receptacle_GCT_USB4105-xx-A_16P_TopMnt_Horizontal; LCSC Part Number C165948 -> (none)
Connections:
- net +3V3: now also C3.1, R2.2, R3.2, U1.20 (VCC), U1.4 (VCCIO)
- net DTR: now also U1.2 (DTR)
- net GND: now also C1.2, C3.2, U1.18 (GND), U1.21 (GND), U1.25 (AGND), U1.26 (TEST), U1.7 (GND)
- net RTS: now also U1.3 (RTS)
- net RX: now also U1.1 (TXD)
- net TX: now also U1.5 (RXD)
- net USBD+: now also U1.15 (USBD+)
- net USBD-: now also U1.16 (USBD-)
- new net: D2.2 (A), R3.1
- new net: D2.1 (K), U1.23 (CBUS0)
- new net: C1.1, U1.17 (3V3OUT), U1.19 (~{RESET})
- new net: D1.2 (A), R2.1
- new net: D1.1 (K), U1.22 (CBUS1)
- no-connect marks 14 -> 22
Other:
- moved on the sheet: C2, C5, C6, R7, R8, U3, USB1
